File: ECAD/LFO Small.brd (EAGLE design)
At the start: 81.8 x 43.5 mm, 14 parts

Commit message: Removed external Eagle library dependencies.
Parts:
- D2: device My Components:LED_BARGRAPH_6 -> SynthLib:LED_BARGRAPH_6
- L1, L2, L3: device adafruit:WS2812B -> SynthLib:WS2812B
- S1: device SparkFun-Electromechanical:TACTILE-PTH-12MM -> SynthLib:TACTILE-PTH-12MM
- S2, S3: device SparkFun-Electromechanical:TACTILE-SWITCH-SMD -> SynthLib:TACTILE-SWITCH-SMD
- U$1: device TeensyLC:TEENSY_LC_BASIC -> SynthLib:TEENSY_LC_BASIC
- U$2, U$3: device My Components:14MMPOT -> SynthLib:14MMPOT
- U$5: device My Components:MEZZ -> SynthLib:MEZZ
Routing:
- net GND: track 23.5 -> 38.6 mm
- net N$13: track 91.1 -> 99.9 mm
- net N$16: track 100.6 -> 106.4 mm
Changed lines of the file:
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@@
 </class>
 </classes>
-<designrules name="default *">
+<designrules name="LaenPCBOrder *">
 <description language="de">&lt;b&gt;EAGLE Design Rules&lt;/b&gt;
 &lt;p&gt;
@@
 Einstellungen hier und speichern die Design Rules unter
 einem neuen Namen ab.</description>
-<description language="en">&lt;b&gt;EAGLE Design Rules&lt;/b&gt;
+<description language="en">&lt;b&gt;Laen's PCB Order Design Rules&lt;/b&gt;
 &lt;p&gt;
-The default Design Rules have been set to cover
-a wide range of applications. Your particular design
-may have different requirements, so please make the
-necessary adjustments and save your customized
-design rules under a new name.</description>
+Please make sure your boards conform to these design rules.</description>
 <param name="layerSetup" value="(1*16)"/>
-<param name="mtCopper" value="0.035mm 0.035mm 0.035mm 0.035mm 0.035mm 0.035mm 0.035mm 0.035mm 0.035mm 0.035mm 0.035mm 0.035mm 0.035mm 0.035mm 0.035mm 0.035mm"/>
-<param name="mtIsolate" value="1.5mm 0.15mm 0.2mm 0.15mm 0.2mm 0.15mm 0.2mm 0.15mm 0.2mm 0.15mm 0.2mm 0.15mm 0.2mm 0.15mm 0.2mm"/>
-<param name="mdWireWire" value="8mil"/>
-<param name="mdWirePad" value="8mil"/>
-<param name="mdWireVia" value="8mil"/>
-<param name="mdPadPad" value="8mil"/>
-<param name="mdPadVia" value="8mil"/>
-<param name="mdViaVia" value="8mil"/>
-<param name="mdSmdPad" value="8mil"/>
-<param name="mdSmdVia" value="8mil"/>
-<param name="mdSmdSmd" value="8mil"/>
+<param name="mtCopper" value="0.0356mm 0.0356mm 0.0356mm 0.0356mm 0.0356mm 0.0356mm 0.0356mm 0.0356mm 0.0356mm 0.0356mm 0.0356mm 0.0356mm 0.0356mm 0.0356mm 0.0356mm 0.0356mm"/>
+<param name="mtIsolate" value="1.5011mm 0.1499mm 0.2007mm 0.1499mm 0.2007mm 0.1499mm 0.2007mm 0.1499mm 0.2007mm 0.1499mm 0.2007mm 0.1499mm 0.2007mm 0.1499mm 0.2007mm"/>
+<param name="mdWireWire" value="6mil"/>
+<param name="mdWirePad" value="6mil"/>
+<param name="mdWireVia" value="6mil"/>
+<param name="mdPadPad" value="6mil"/>
+<param name="mdPadVia" value="6mil"/>
+<param name="mdViaVia" value="6mil"/>
+<param name="mdSmdPad" value="6mil"/>
+<param name="mdSmdVia" value="6mil"/>
+<param name="mdSmdSmd" value="6mil"/>
 <param name="mdViaViaSameLayer" value="8mil"/>
 <param name="mnLayersViaInSmd" value="2"/>
-<param name="mdCopperDimension" value="25mil"/>
-<param name="mdDrill" value="8mil"/>
+<param name="mdCopperDimension" value="15mil"/>
+<param name="mdDrill" value="6mil"/>
 <param name="mdSmdStop" value="0mil"/>
-<param name="msWidth" value="10mil"/>
+<param name="msWidth" value="6mil"/>
 <param name="msDrill" value="13mil"/>
-<param name="msMicroVia" value="9.99mm"/>
+<param name="msMicroVia" value="13mil"/>
 <param name="msBlindViaRatio" value="0.5"/>
 <param name="rvPadTop" value="0.25"/>
@@
 <param name="rvMicroViaOuter" value="0.25"/>
 <param name="rvMicroViaInner" value="0.25"/>
-<param name="rlMinPadTop" value="10mil"/>
+<param name="rlMinPadTop" value="7mil"/>
 <param name="rlMaxPadTop" value="20mil"/>
-<param name="rlMinPadInner" value="10mil"/>
+<param name="rlMinPadInner" value="7mil"/>
 <param name="rlMaxPadInner" value="20mil"/>
-<param name="rlMinPadBottom" value="10mil"/>
+<param name="rlMinPadBottom" value="7mil"/>
 <param name="rlMaxPadBottom" value="20mil"/>
-<param name="rlMinViaOuter" value="8mil"/>
+<param name="rlMinViaOuter" value="7mil"/>
 <param name="rlMaxViaOuter" value="20mil"/>
-<param name="rlMinViaInner" value="8mil"/>
+<param name="rlMinViaInner" value="7mil"/>
 <param name="rlMaxViaInner" value="20mil"/>
 <param name="rlMinMicroViaOuter" value="4mil"/>
@@
 <param name="mvStopFrame" value="1"/>
 <param name="mvCreamFrame" value="0"/>
-<param name="mlMinStopFrame" value="4mil"/>
-<param name="mlMaxStopFrame" value="4mil"/>
+<param name="mlMinStopFrame" value="3mil"/>
+<param name="mlMaxStopFrame" value="3mil"/>
 <param name="mlMinCreamFrame" value="0mil"/>
 <param name="mlMaxCreamFrame" value="0mil"/>
@@
 <attribute name="NAME" x="3.361" y="41.309" size="1.27" layer="26" ratio="10" rot="MR270"/>
 </element>
-<element name="L1" library="adafruit" package="WS2812B" value="WS2812B" x="20.65" y="5.55833125" rot="R90"/>
-<element name="L2" library="adafruit" package="WS2812B" value="WS2812B" x="32.25" y="24.451"/>
-<element name="L3" library="adafruit" package="WS2812B" value="WS2812B" x="53.75" y="24.451"/>
-<element name="U$1" library="TeensyLC" package="TEENSY_LC_BASIC" value="TEENSY_LC_BASIC" x="9.08" y="19.05" smashed="yes" rot="MR180">
+<element name="L1" library="SynthLib" package="WS2812B" value="WS2812B" x="20.65" y="5.55833125" rot="R90"/>
+<element name="L2" library="SynthLib" package="WS2812B" value="WS2812B" x="32.25" y="24.451"/>
+<element name="L3" library="SynthLib" package="WS2812B" value="WS2812B" x="53.75" y="24.451"/>
+<element name="U$1" library="SynthLib" package="TEENSY_LC_BASIC" value="TEENSY_LC_BASIC" x="9.08" y="19.05" smashed="yes" rot="MR180">
 <attribute name="NAME" x="6.54" y="5.08" size="1.27" layer="26" font="vector" rot="MR180"/>
 </element>
-<element name="U$2" library="My Components" package="14MMPOT" value="10K" x="32.25" y="24.451"/>
-<element name="U$3" library="My Components" package="14MMPOT" value="10K" x="53.75" y="24.451"/>
-<element name="U$5" library="My Components" package="MEZZ" value="TL1220MEZZ" x="75.25" y="24.451" rot="R90"/>
-<element name="S3" library="SparkFun-Electromechanical" package="TACTILE-SWITCH-SMD" value="SWITCH-MOMENTARY-2SMD" x="53.75" y="7" smashed="yes" rot="MR0">
+<element name="U$2" library="SynthLib" package="14MMPOT" value="10K" x="32.25" y="24.451"/>
+<element name="U$3" library="SynthLib" package="14MMPOT" value="10K" x="53.75" y="24.451"/>
+<element name="U$5" library="SynthLib" package="MEZZ" value="TL1220MEZZ" x="75.25" y="24.451" rot="R90"/>
+<element name="S3" library="SynthLib" package="TACTILE-SWITCH-SMD" value="SWITCH-MOMENTARY-2SMD" x="53.75" y="7" smashed="yes" rot="MR0">
 <attribute name="PROD_ID" value="SWCH-08247" x="53.75" y="7" size="1.778" layer="28" rot="MR0" display="off"/>
 <attribute name="NAME" x="54.639" y="8.778" size="0.4064" layer="26" rot="MR0"/>
 </element>
-<element name="D2" library="My Components" package="LED_BARGRAPH_6" value="Blue" x="7.08" y="25.471" rot="R270"/>
-<element name="S1" library="SparkFun-Electromechanical" package="TACTILE-PTH-12MM" value="SWITCH-MOMENTARY-212MM" x="9.035" y="7.451040625" rot="R90">
+<element name="D2" library="SynthLib" package="LED_BARGRAPH_6" value="Blue" x="7.08" y="25.471" rot="R270"/>
+<element name="S1" library="SynthLib" package="TACTILE-PTH-12MM" value="SWITCH-MOMENTARY-212MM" x="9.035" y="7.451040625" rot="R90">
 <attribute name="PROD_ID" value="SWCH-09185" x="9.035" y="7.451040625" size="1.778" layer="27" rot="R90" display="off"/>
 </element>
-<element name="S2" library="SparkFun-Electromechanical" package="TACTILE-SWITCH-SMD" value="SWITCH-MOMENTARY-2SMD" x="32.25" y="7" smashed="yes" rot="MR180">
+<element name="S2" library="SynthLib" package="TACTILE-SWITCH-SMD" value="SWITCH-MOMENTARY-2SMD" x="32.25" y="7" smashed="yes" rot="MR180">
 <attribute name="PROD_ID" value="SWCH-08247" x="32.25" y="7" size="1.778" layer="28" rot="MR180" display="off"/>
 <attribute name="NAME" x="31.361" y="5.222" size="0.4064" layer="26" rot="MR180"/>
@@
 <wire x1="19" y1="3.144790625" x2="18.92560625" y2="3.32439375" width="0.254" layer="1" curve="44.999502"/>
 <wire x1="18.92560625" y1="3.32439375" x2="18.75" y2="3.5" width="0.254" layer="1"/>
-<wire x1="11.46060625" y1="12.54060625" x2="11.535" y2="12.720209375" width="0.254" layer="16" curve="44.999295"/>
 <contactref element="U$1" pad="GND2"/>
 <contactref element="U$2" pad="P$5"/>
@@
 <wire x1="9.08" y1="35.56" x2="9.69" y2="35.56" width="0.6096" layer="16"/>
 <wire x1="9.69" y1="35.56" x2="10.89" y2="34.36" width="0.6096" layer="16"/>
-<wire x1="11.535" y1="13.701040625" x2="11.535" y2="12.720209375" width="0" layer="19" extent="16-16"/>
-<wire x1="1.46" y1="2.54" x2="11.46060625" y2="12.54060625" width="0" layer="19" extent="16-16"/>
+<wire x1="11.535" y1="13.701040625" x2="11.535" y2="12.615" width="0.4064" layer="16"/>
+<wire x1="11.535" y1="12.615" x2="1.46" y2="2.54" width="0.4064" layer="16"/>
 </signal>
 <signal name="N$1">
@@
 <wire x1="74" y1="30.5" x2="74" y2="29.551" width="0.254" layer="16"/>
 <wire x1="74" y1="29.551" x2="73.98" y2="29.531" width="0.254" layer="16"/>
+<wire x1="73.98" y1="29.531" x2="73.98" y2="28.769" width="0.4064" layer="16"/>
+<wire x1="73.98" y1="28.769" x2="72.202" y2="26.991" width="0.4064" layer="16"/>
+<wire x1="73.98" y1="29.531" x2="73.98" y2="29.27" width="0.4064" layer="16"/>
+<wire x1="73.98" y1="29.27" x2="76.25" y2="27" width="0.4064" layer="16"/>
+<wire x1="76.25" y1="27" x2="78.289" y2="27" width="0.4064" layer="16"/>
+<wire x1="78.289" y1="27" x2="78.298" y2="26.991" width="0.4064" layer="16"/>
 </signal>
 <signal name="3.3V">
@@
 <wire x1="18.5" y1="41.75" x2="15.5" y2="38.75" width="0.254" layer="16"/>
 <via x="15.5" y="38.75" extent="1-16" drill="0.5"/>
+<wire x1="73.98" y1="19.371" x2="73.98" y2="22.673" width="0.4064" layer="16"/>
+<wire x1="73.98" y1="22.673" x2="72.202" y2="24.451" width="0.4064" layer="16"/>
 </signal>
 <signal name="N$18">
