File: ECAD/LFO Small.sch (EAGLE design)
At the start: 12 parts

Commit message: Removed external Eagle library dependencies.
Parts:
- D2: device My Components:LED_BARGRAPH_6 -> SynthLib:LED_BARGRAPH_6
- L1, L2, L3: device adafruit:WS2812B -> SynthLib:WS2812B
- S1: device SparkFun-Electromechanical:SWITCH-MOMENTARY-212MM -> SynthLib:SWITCH-MOMENTARY-212MM
- S2, S3: device SparkFun-Electromechanical:SWITCH-MOMENTARY-2SMD -> SynthLib:SWITCH-MOMENTARY-2SMD
- U$1: device TeensyLC:TEENSY_LC_BASIC -> SynthLib:TEENSY_LC_BASIC
- U$2, U$3: device My Components:ALPHA1400F10K -> SynthLib:ALPHA1400F10K
- U$5: device My Components:TL1220MEZZ -> SynthLib:TL1220MEZZ
Changed lines of the file:
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@@
 </classes>
 <parts>
-<part name="U$1" library="TeensyLC" deviceset="TEENSY_LC_BASIC" device=""/>
+<part name="U$1" library="SynthLib" deviceset="TEENSY_LC_BASIC" device=""/>
 <part name="FRAME1" library="frames" deviceset="LETTER_L" device="" value="asdf"/>
-<part name="L1" library="adafruit" deviceset="WS2812B" device=""/>
-<part name="L2" library="adafruit" deviceset="WS2812B" device=""/>
-<part name="L3" library="adafruit" deviceset="WS2812B" device=""/>
-<part name="U$2" library="My Components" deviceset="ALPHA1400F" device="10K" value="10K"/>
-<part name="U$3" library="My Components" deviceset="ALPHA1400F" device="10K" value="10K"/>
-<part name="U$5" library="My Components" deviceset="TL1220MEZZ" device=""/>
+<part name="L1" library="SynthLib" deviceset="WS2812B" device=""/>
+<part name="L2" library="SynthLib" deviceset="WS2812B" device=""/>
+<part name="L3" library="SynthLib" deviceset="WS2812B" device=""/>
+<part name="U$2" library="SynthLib" deviceset="ALPHA1400F" device="10K" value="10K"/>
+<part name="U$3" library="SynthLib" deviceset="ALPHA1400F" device="10K" value="10K"/>
+<part name="U$5" library="SynthLib" deviceset="TL1220MEZZ" device=""/>
 <part name="JP1" library="jumper" deviceset="JP3Q" device="" value="JP1"/>
-<part name="S3" library="SparkFun-Electromechanical" deviceset="SWITCH-MOMENTARY-2" device="SMD"/>
-<part name="D2" library="My Components" deviceset="LED_BARGRAPH_6" device="" value="Blue"/>
-<part name="S1" library="SparkFun-Electromechanical" deviceset="SWITCH-MOMENTARY-2" device="12MM"/>
-<part name="S2" library="SparkFun-Electromechanical" deviceset="SWITCH-MOMENTARY-2" device="SMD"/>
-<part name="GND4" library="My Components" deviceset="GND2" device=""/>
-<part name="GND5" library="My Components" deviceset="GND2" device=""/>
-<part name="GND6" library="My Components" deviceset="GND2" device=""/>
-<part name="GND7" library="My Components" deviceset="GND2" device=""/>
-<part name="GND1" library="My Components" deviceset="GND2" device=""/>
-<part name="GND2" library="My Components" deviceset="GND2" device=""/>
-<part name="GND3" library="My Components" deviceset="GND2" device=""/>
-<part name="GND8" library="My Components" deviceset="GND2" device=""/>
-<part name="GND9" library="My Components" deviceset="GND2" device=""/>
-<part name="GND10" library="My Components" deviceset="GND2" device=""/>
-<part name="GND11" library="My Components" deviceset="GND2" device=""/>
+<part name="S3" library="SynthLib" deviceset="SWITCH-MOMENTARY-2" device="SMD"/>
+<part name="D2" library="SynthLib" deviceset="LED_BARGRAPH_6" device="" value="Blue"/>
+<part name="S1" library="SynthLib" deviceset="SWITCH-MOMENTARY-2" device="12MM"/>
+<part name="S2" library="SynthLib" deviceset="SWITCH-MOMENTARY-2" device="SMD"/>
+<part name="GND4" library="SynthLib" deviceset="GND2" device=""/>
+<part name="GND5" library="SynthLib" deviceset="GND2" device=""/>
+<part name="GND6" library="SynthLib" deviceset="GND2" device=""/>
+<part name="GND7" library="SynthLib" deviceset="GND2" device=""/>
+<part name="GND1" library="SynthLib" deviceset="GND2" device=""/>
+<part name="GND2" library="SynthLib" deviceset="GND2" device=""/>
+<part name="GND3" library="SynthLib" deviceset="GND2" device=""/>
+<part name="GND8" library="SynthLib" deviceset="GND2" device=""/>
+<part name="GND9" library="SynthLib" deviceset="GND2" device=""/>
+<part name="GND10" library="SynthLib" deviceset="GND2" device=""/>
+<part name="GND11" library="SynthLib" deviceset="GND2" device=""/>
 </parts>
 <sheets>
