File: ECAD/Filter.brd (EAGLE design)
At the start: 104 x 43.5 mm, 22 parts

Commit message: Moved the LED bar graphs' color labels to the silkscreen layer.
Changed lines of the file:
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@@
 <elements>
 <element name="D1" library="SynthLib" package="LED_BARGRAPH_6" value="Red" x="7.08" y="25.471" smashed="yes" rot="R270">
-<attribute name="VALUE" x="5.611665625" y="26.867665625" size="1.27" layer="27"/>
+<attribute name="VALUE" x="5.611665625" y="26.867665625" size="1.27" layer="21"/>
 </element>
 <element name="JP1" library="jumper" package="JP3Q" value="SPI_POWER" x="7.67" y="39.603334375" smashed="yes" rot="MR180"/>
