File: ECAD/Oscillator.sch (EAGLE design)
At the start: 14 parts

Commit message: Moved the LED bar graphs' color labels to the silkscreen layer.
Parts:
- D1: value Red -> Amber
Changed lines of the file:
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@@
 <part name="U$1" library="SynthLib" deviceset="TEENSY_LC_BASIC" device=""/>
 <part name="JP1" library="jumper" deviceset="JP3Q" device="" value="SPI_POWER"/>
-<part name="D1" library="SynthLib" deviceset="LED_BARGRAPH_6" device="" value="Red"/>
+<part name="D1" library="SynthLib" deviceset="LED_BARGRAPH_6" device="" value="Amber"/>
 <part name="GND1" library="SynthLib" deviceset="GND2" device=""/>
 <part name="GND2" library="SynthLib" deviceset="GND2" device=""/>
