File: ECAD/Envelope.brd (EAGLE design)
At the start: 129 x 43.5 mm, 15 parts

Commit message: Designed the Envelope board.  Fairly straightforward, except that it has three variants.
Parts:
- added JP2: Master Volume, SynthLib:JP3Q
- added U$10, U$11, U$12, U$8, U$9: (no value), SynthLib:STANDOFF-M3
- JP1: value SPI_POWER -> SPI
- moved JP1 118.9 mm to (51.4, 6.27)
- moved L7 95.1 mm to (42.1, 5.56), turned to 90 degrees
- moved U$1 46.1 mm to (101.8, 10.1), flipped to the bottom, turned to 90 degrees
- turned L2 to 180 degrees
- turned L3 to 180 degrees
- turned L4 to 180 degrees
- turned L5 to 180 degrees
- turned L6 to 180 degrees
Connections:
- new net N$12: JP2.6, U$1.5
- net 3.3V: now also JP2.3; no longer U$1.3.3V
- net GND: now also JP2.5
- net N$26: now also JP2.2
- net N$27: now also JP2.4
- net VIN: now also JP2.1
Routing:
- net N$2: track 0.00 -> 171.2 mm
- net VIN: track 0.00 -> 160.4 mm
- net N$6: track 0.00 -> 125.3 mm
- net N$11: track 0.00 -> 118.8 mm
- net N$27: track 0.00 -> 118.4 mm
- net 3.3V: track 0.00 -> 110.4 mm
- net N$1: track 0.00 -> 99.0 mm
- net N$26: track 0.00 -> 63.1 mm
- net N$10: track 0.00 -> 49.1 mm
- net N$28: track 0.00 -> 42.0 mm
- net N$12: track 0.00 -> 40.7 mm
- net N$23: track 0.00 -> 40.3 mm
- net N$24: track 0.00 -> 37.5 mm
- net N$21: track 0.00 -> 37.5 mm
- net N$7: track 0.00 -> 37.3 mm
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- added copper zone on layer 1, net GND
Other:
- board size 129 x 43.5 mm -> 122.5 x 39 mm
