File: ECAD/io_daughterboard/pcb/io_daughterboard.sch (KiCad schematic (older format))
At the start: 52 parts, among them P1 CONN_02X32, P2 CONN_02X32

Commit message: added slave connectors to schematic; laid out page.
Parts:
- removed P? (x15): CONN_01X06, symbol CONN_01X06
- removed U? (x4): 74HC244, symbol 74HC244
- added P? (x15): CONN_01X06, symbol CONN_01X06
- added R? (x4): 100K, symbol R
- added R? (x4): 4K7, symbol R
- added R? (x20): 10K, symbol R
- added U? (x4): 74HC244, symbol 74HC244
Connections:
- net BTN_RESET is gone; now on net BTN_~RESET: C?.1, R?.2, SW?.1, SW?.3
- net +3V3: now also U?.14 (Vio), U?.20 (Vcc), U?.20 (Vcc), U?.3 (A0/Data_Out), U?.6 (Vcc), R?.1, R?.1, R?.1, R?.1, R?.1, R?.1, R?.1, R?.1, R?.1, R?.1, R?.1, R?.1, R?.1, R?.1, R?.1, R?.1, R?.1, R?.1, R?.1, R?.1, R?.1, R?.1, R?.1, R?.1, U?.20 (Vcc), U?.20 (Vcc), U?.20 (Vcc)
- net +5V: now also P?.2 (P2), P?.2 (P2), P?.2 (P2), P?.2 (P2), P?.2 (P2), P?.2 (P2), P?.2 (P2), P?.2 (P2), P?.2 (P2), P?.2 (P2), P?.2 (P2), P?.2 (P2), P?.2 (P2), P?.2 (P2), P?.2 (P2), P?.2 (P2)
- net GND: now also P?.6 (P6), R?.2, U?.10 (GND), U?.10 (GND), U?.10 (GND), P?.6 (P6), P?.6 (P6), P?.6 (P6), P?.6 (P6), P?.6 (P6), P?.6 (P6), P?.6 (P6), P?.6 (P6), P?.6 (P6), P?.6 (P6), P?.6 (P6), P?.6 (P6), P?.6 (P6), P?.6 (P6), P?.6 (P6), R?.1, R?.1, R?.1, R?.1, U?.10 (GND), U?.10 (GND), U?.10 (GND), U?.10 (GND); no longer R?.1
- net I²C3_SCL: now also U?.4 (SCLK), R?.2
- net I²C3_SDA: now also U?.5 (SDAT), R?.2
- net PA5: now also U?.17 (2A0), U?.17 (2A0), U?.17 (2A0), U?.17 (2A0)
- net PA7: now also U?.17 (2A0), U?.2 (1A0), U?.17 (2A0), U?.2 (1A0)
- net PB3: now also U?.15 (2A1), U?.15 (2A1), U?.15 (2A1), U?.15 (2A1)
- net PB4: now also U?.18 (1Y0), U?.18 (1Y0), U?.18 (1Y0), U?.18 (1Y0)
- net PB7: now also P?.5 (P5), U?.1 (1~OE), U?.1 (1~OE), U?.19 (2~OE), P?.5 (P5), P?.5 (P5), P?.5 (P5), R?.2
- net PC11: now also U?.16 (1Y1), U?.16 (1Y1), U?.16 (1Y1), U?.16 (1Y1)
- net PC12: now also U?.15 (2A1), U?.4 (1A1), U?.15 (2A1), U?.4 (1A1)
- net PC3: now also P?.5 (P5), P?.5 (P5), P?.5 (P5), P?.5 (P5), R?.2, U?.1 (1~OE), U?.1 (1~OE), U?.19 (2~OE)
- net PC8: now also P?.5 (P5), P?.5 (P5), P?.5 (P5), P?.5 (P5), R?.2, U?.1 (1~OE), U?.19 (2~OE), U?.19 (2~OE)
- net PE2: now also U?.13 (2A2), U?.13 (2A2), U?.13 (2A2), U?.13 (2A2)
- net PE3: now also U?.19 (2~OE), P?.5 (P5), P?.5 (P5), P?.5 (P5), P?.5 (P5), R?.2, U?.1 (1~OE), U?.19 (2~OE)
- net PE5: now also U?.14 (1Y2), U?.14 (1Y2), U?.14 (1Y2), U?.14 (1Y2)
- net PE6: now also U?.13 (2A2), U?.6 (1A3), U?.13 (2A2), U?.6 (1A3)
- net PF7: now also U?.11 (2A3), U?.11 (2A3), U?.11 (2A3), U?.11 (2A3)
- net PF8: now also U?.12 (1Y3), U?.12 (1Y3), U?.12 (1Y3), U?.12 (1Y3)
- net PF9: now also U?.11 (2A3), U?.8 (1A3), U?.11 (2A3), U?.8 (1A3)
- net PG2: now also U?.2 (INT), R?.2
- net RTOUCH_XL: now also U?.16 (X-)
- net RTOUCH_XR: now also U?.13 (X+)
- net RTOUCH_YD: now also U?.1 (Y-)
- net RTOUCH_YU: now also U?.15 (Y+)
- net at U?.11 (IN2): now also R?.2
- net at U?.12 (IN3): now also R?.2
- net at U?.7 (Data_In): now also R?.2
- net at U?.8 (IN0): now also R?.2
- net at U?.9 (IN1): now also R?.2
- net SLV1A_MISO: now reaches P?.1 (P1)
- net SLV1A_MISO: now also U?.2 (1A0), R?.2
- net SLV1A_SCK: now reaches P?.3 (P3)
- net SLV1A_SCK: now also U?.3 (2Y0)
- net SLV1A_MOSI: now reaches P?.4 (P4)
- net SLV3A_MISO: now reaches U?.4 (1A1)
- net SLV3A_MISO: now also P?.1 (P1), R?.2
- net SLV3A_SCK: now reaches U?.5 (2Y1)
- net SLV3A_SCK: now also P?.3 (P3)
- net SLV4A_MISO: now reaches U?.6 (1A3)
- net SLV4A_MISO: now also P?.1 (P1), R?.2
- net SLV4A_SCK: now reaches U?.7 (2Y2)
- net SLV4A_SCK: now also P?.3 (P3)
- net SLV5A_MISO: now reaches U?.8 (1A3)
- net SLV5A_MISO: now also R?.2
- net SLV5A_SCK: now reaches U?.9 (2Y3)
- net SLV5A_SCK: now also P?.3 (P3)
- net at SW?.2, SW?.4: now also R?.1; no longer R?.2
- new net SLV1B_MISO: P?.1 (P1), R?.2, U?.2 (1A0)
- new net SLV1B_MOSI: P?.4 (P4)
- new net SLV1B_SCK: P?.3 (P3), U?.3 (2Y0)
- new net SLV1C_MISO: P?.1 (P1), R?.2, U?.2 (1A0)
- new net SLV1C_MOSI: P?.4 (P4)
- new net SLV1C_SCK: P?.3 (P3), U?.3 (2Y0)
- new net SLV1D_MISO: P?.1 (P1), R?.2, U?.2 (1A0)
- new net SLV1D_MOSI: P?.4 (P4)
- new net SLV1D_SCK: P?.3 (P3), U?.3 (2Y0)
- new net SLV3A_MOSI: P?.4 (P4)
- new net SLV3B_MISO: P?.1 (P1), R?.2, U?.4 (1A1)
- new net SLV3B_MOSI: P?.4 (P4)
- new net SLV3B_SCK: P?.3 (P3), U?.5 (2Y1)
- new net SLV3C_MISO: P?.1 (P1), R?.2, U?.4 (1A1)
- new net SLV3C_MOSI: P?.4 (P4)
- new net SLV3C_SCK: P?.3 (P3), U?.5 (2Y1)
- new net SLV3D_MISO: P?.1 (P1), R?.2, U?.4 (1A1)
- new net SLV3D_MOSI: P?.4 (P4)
- new net SLV3D_SCK: P?.3 (P3), U?.5 (2Y1)
- new net SLV4A_MOSI: P?.4 (P4)
- new net SLV4B_MISO: P?.1 (P1), R?.2, U?.6 (1A3)
- new net SLV4B_MOSI: P?.4 (P4)
- new net SLV4B_SCK: P?.3 (P3), U?.7 (2Y2)
- new net SLV4C_MISO: P?.1 (P1), R?.2, U?.6 (1A3)
- new net SLV4C_MOSI: P?.4 (P4)
- new net SLV4C_SCK: P?.3 (P3), U?.7 (2Y2)
- new net SLV4D_MISO: P?.1 (P1), R?.2, U?.6 (1A3)
- new net SLV4D_MOSI: P?.4 (P4)
- new net SLV4D_SCK: P?.3 (P3), U?.7 (2Y2)
- new net SLV5A_MISO_Fred: P?.1 (P1)
- new net SLV5A_MOSI: P?.4 (P4)
- new net SLV5B_MISO: P?.1 (P1), R?.2, U?.8 (1A3)
- new net SLV5B_MOSI: P?.4 (P4)
- new net SLV5B_SCK: P?.3 (P3), U?.9 (2Y3)
- new net SLV5C_MISO: P?.1 (P1), R?.2, U?.8 (1A3)
- new net SLV5C_MOSI: P?.4 (P4)
- new net SLV5C_SCK: P?.3 (P3), U?.9 (2Y3)
- new net SLV5D_MISO: P?.1 (P1), R?.2, U?.8 (1A3)
- new net SLV5D_MOSI: P?.4 (P4)
- new net SLV5D_SCK: P?.3 (P3), U?.9 (2Y3)
Other:
- note added: "Master Interface"
- note added: "SPI Crossbar"
- note added: "Slave Interfaces"
- note removed: "Backlight Power"
- note removed: "Master"
- note removed: "SPI Routing"
- note removed: "Slaves"
- moved on the sheet: C?, CON?, D?, J?, L?, P1, P2, P?, R?, SW?, U?
