File: ECAD/io_daughterboard/pcb/io_daughterboard.sch (KiCad schematic (older format))
At the start: 89 parts, among them CON1 BARREL_JACK, J1 XF2L-0625-1A, J2 4-1734839-0, P1 CONN_02X32, P10 Slave 5B, P11 Slave 1C, P12 Slave 3C, P13 Slave 4C, P14 Slave 5C, P15 Slave 1D, P16 Slave 3D, P17 Slave 4D, P18 Slave 5D, P19 CONN_01X04, P2 CONN_02X32, P3 Slave 1A, P4 Slave 3A, P5 Slave 4A, P6 Slave 5A, P7 Slave 1B, P8 Slave 3B, P9 Slave 4B, SW1 Reset Button, SW2 User Button, U1 FAN5333BSX, U10 SN74LV1T34DCKR, U11 SN74LV1T34DCKR, U2 SPX3819M5-L-3-3, U3 74HC244, U4 74HC244, U5 74HC244, U6 STMPE811QTR, U7 74HC244, U8 74HC244, U9 74HC244

Commit message: P1 and P2 connectors placed.  Back to PicoBlade through-hole connectors.
Parts:
- P10, P11, P12, P13, P14, P15, P16, P17, P18, P3, P4, P5, P6, P7, P8, P9: footprint Pin_Headers:Pin_Header_Straight_2x03_Pitch2.00mm -> Connectors_Molex:Molex_PicoBlade_53047-0610_06x1.25mm_Straight
- P19: footprint daughterfeet:B4B-PH-SM4-TB -> Connectors_Molex:Molex_PicoBlade_53047-0410_04x1.25mm_Straight
Changed lines of the file:
@@
 F 0 "P3" H 1750 5850 50  0000 C CNN
 F 1 "Slave 1A" V 1850 5500 50  0000 C CNN
-F 2 "Pin_Headers:Pin_Header_Straight_2x03_Pitch2.00mm" H 1750 5500 50  0001 C CNN
+F 2 "Connectors_Molex:Molex_PicoBlade_53047-0610_06x1.25mm_Straight" H 1750 5500 50  0001 C CNN
 F 3 "" H 1750 5500 50  0000 C CNN
 	1    1750 5500
@@
 F 0 "P19" H 16050 8050 50  0000 C CNN
 F 1 "CONN_01X04" V 16150 7800 50  0000 C CNN
-F 2 "daughterfeet:B4B-PH-SM4-TB" H 16050 7800 50  0001 C CNN
+F 2 "Connectors_Molex:Molex_PicoBlade_53047-0410_04x1.25mm_Straight" H 16050 7800 50  0001 C CNN
 F 3 "" H 16050 7800 50  0000 C CNN
 	1    16050 7800
@@
 F 0 "P7" H 3150 5850 50  0000 C CNN
 F 1 "Slave 1B" V 3250 5500 50  0000 C CNN
-F 2 "Pin_Headers:Pin_Header_Straight_2x03_Pitch2.00mm" H 3150 5500 50  0001 C CNN
+F 2 "Connectors_Molex:Molex_PicoBlade_53047-0610_06x1.25mm_Straight" H 3150 5500 50  0001 C CNN
 F 3 "" H 3150 5500 50  0000 C CNN
 	1    3150 5500
@@
 F 0 "P11" H 4550 5850 50  0000 C CNN
 F 1 "Slave 1C" V 4650 5500 50  0000 C CNN
-F 2 "Pin_Headers:Pin_Header_Straight_2x03_Pitch2.00mm" H 4550 5500 50  0001 C CNN
+F 2 "Connectors_Molex:Molex_PicoBlade_53047-0610_06x1.25mm_Straight" H 4550 5500 50  0001 C CNN
 F 3 "" H 4550 5500 50  0000 C CNN
 	1    4550 5500
@@
 F 0 "P4" H 1750 6850 50  0000 C CNN
 F 1 "Slave 3A" V 1850 6500 50  0000 C CNN
-F 2 "Pin_Headers:Pin_Header_Straight_2x03_Pitch2.00mm" H 1750 6500 50  0001 C CNN
+F 2 "Connectors_Molex:Molex_PicoBlade_53047-0610_06x1.25mm_Straight" H 1750 6500 50  0001 C CNN
 F 3 "" H 1750 6500 50  0000 C CNN
 	1    1750 6500
@@
 F 0 "P8" H 3150 6850 50  0000 C CNN
 F 1 "Slave 3B" V 3250 6500 50  0000 C CNN
-F 2 "Pin_Headers:Pin_Header_Straight_2x03_Pitch2.00mm" H 3150 6500 50  0001 C CNN
+F 2 "Connectors_Molex:Molex_PicoBlade_53047-0610_06x1.25mm_Straight" H 3150 6500 50  0001 C CNN
 F 3 "" H 3150 6500 50  0000 C CNN
 	1    3150 6500
@@
 F 0 "P12" H 4550 6850 50  0000 C CNN
 F 1 "Slave 3C" V 4650 6500 50  0000 C CNN
-F 2 "Pin_Headers:Pin_Header_Straight_2x03_Pitch2.00mm" H 4550 6500 50  0001 C CNN
+F 2 "Connectors_Molex:Molex_PicoBlade_53047-0610_06x1.25mm_Straight" H 4550 6500 50  0001 C CNN
 F 3 "" H 4550 6500 50  0000 C CNN
 	1    4550 6500
@@
 F 0 "P15" H 5950 5850 50  0000 C CNN
 F 1 "Slave 1D" V 6050 5500 50  0000 C CNN
-F 2 "Pin_Headers:Pin_Header_Straight_2x03_Pitch2.00mm" H 5950 5500 50  0001 C CNN
+F 2 "Connectors_Molex:Molex_PicoBlade_53047-0610_06x1.25mm_Straight" H 5950 5500 50  0001 C CNN
 F 3 "" H 5950 5500 50  0000 C CNN
 	1    5950 5500
@@
 F 0 "P16" H 5950 6850 50  0000 C CNN
 F 1 "Slave 3D" V 6050 6500 50  0000 C CNN
-F 2 "Pin_Headers:Pin_Header_Straight_2x03_Pitch2.00mm" H 5950 6500 50  0001 C CNN
+F 2 "Connectors_Molex:Molex_PicoBlade_53047-0610_06x1.25mm_Straight" H 5950 6500 50  0001 C CNN
 F 3 "" H 5950 6500 50  0000 C CNN
 	1    5950 6500
@@
 F 0 "P5" H 1750 7850 50  0000 C CNN
 F 1 "Slave 4A" V 1850 7500 50  0000 C CNN
-F 2 "Pin_Headers:Pin_Header_Straight_2x03_Pitch2.00mm" H 1750 7500 50  0001 C CNN
+F 2 "Connectors_Molex:Molex_PicoBlade_53047-0610_06x1.25mm_Straight" H 1750 7500 50  0001 C CNN
 F 3 "" H 1750 7500 50  0000 C CNN
 	1    1750 7500
@@
 F 0 "P9" H 3150 7850 50  0000 C CNN
 F 1 "Slave 4B" V 3250 7500 50  0000 C CNN
-F 2 "Pin_Headers:Pin_Header_Straight_2x03_Pitch2.00mm" H 3150 7500 50  0001 C CNN
+F 2 "Connectors_Molex:Molex_PicoBlade_53047-0610_06x1.25mm_Straight" H 3150 7500 50  0001 C CNN
 F 3 "" H 3150 7500 50  0000 C CNN
 	1    3150 7500
@@
 F 0 "P13" H 4550 7850 50  0000 C CNN
 F 1 "Slave 4C" V 4650 7500 50  0000 C CNN
-F 2 "Pin_Headers:Pin_Header_Straight_2x03_Pitch2.00mm" H 4550 7500 50  0001 C CNN
+F 2 "Connectors_Molex:Molex_PicoBlade_53047-0610_06x1.25mm_Straight" H 4550 7500 50  0001 C CNN
 F 3 "" H 4550 7500 50  0000 C CNN
 	1    4550 7500
@@
 F 0 "P6" H 1750 8850 50  0000 C CNN
 F 1 "Slave 5A" V 1850 8500 50  0000 C CNN
-F 2 "Pin_Headers:Pin_Header_Straight_2x03_Pitch2.00mm" H 1750 8500 50  0001 C CNN
+F 2 "Connectors_Molex:Molex_PicoBlade_53047-0610_06x1.25mm_Straight" H 1750 8500 50  0001 C CNN
 F 3 "" H 1750 8500 50  0000 C CNN
 	1    1750 8500
@@
 F 0 "P10" H 3150 8850 50  0000 C CNN
 F 1 "Slave 5B" V 3250 8500 50  0000 C CNN
-F 2 "Pin_Headers:Pin_Header_Straight_2x03_Pitch2.00mm" H 3150 8500 50  0001 C CNN
+F 2 "Connectors_Molex:Molex_PicoBlade_53047-0610_06x1.25mm_Straight" H 3150 8500 50  0001 C CNN
 F 3 "" H 3150 8500 50  0000 C CNN
 	1    3150 8500
@@
 F 0 "P14" H 4550 8850 50  0000 C CNN
 F 1 "Slave 5C" V 4650 8500 50  0000 C CNN
-F 2 "Pin_Headers:Pin_Header_Straight_2x03_Pitch2.00mm" H 4550 8500 50  0001 C CNN
+F 2 "Connectors_Molex:Molex_PicoBlade_53047-0610_06x1.25mm_Straight" H 4550 8500 50  0001 C CNN
 F 3 "" H 4550 8500 50  0000 C CNN
 	1    4550 8500
@@
 F 0 "P17" H 5950 7850 50  0000 C CNN
 F 1 "Slave 4D" V 6050 7500 50  0000 C CNN
-F 2 "Pin_Headers:Pin_Header_Straight_2x03_Pitch2.00mm" H 5950 7500 50  0001 C CNN
+F 2 "Connectors_Molex:Molex_PicoBlade_53047-0610_06x1.25mm_Straight" H 5950 7500 50  0001 C CNN
 F 3 "" H 5950 7500 50  0000 C CNN
 	1    5950 7500
@@
 F 0 "P18" H 5950 8850 50  0000 C CNN
 F 1 "Slave 5D" V 6050 8500 50  0000 C CNN
-F 2 "Pin_Headers:Pin_Header_Straight_2x03_Pitch2.00mm" H 5950 8500 50  0001 C CNN
+F 2 "Connectors_Molex:Molex_PicoBlade_53047-0610_06x1.25mm_Straight" H 5950 8500 50  0001 C CNN
 F 3 "" H 5950 8500 50  0000 C CNN
 	1    5950 8500

Commit message: Moved BARREL_JACK and PicoBlade 4x1 footprints into local library.
Parts:
- CON1: footprint Connect:BARREL_JACK -> daughterfeet:BARREL_JACK
- P10, P11, P12, P13, P14, P15, P16, P17, P18, P3, P4, P5, P6, P7, P8, P9: footprint Connectors_Molex:Molex_PicoBlade_53047-0610_06x1.25mm_Straight -> daughterfeet:Molex_PicoBlade_53047-0610_06x1.25mm_Straight
Connections:
- net PA5: now also U9.17 (2A0), U9.2 (1A0); no longer U7.17 (2A0)
- net PA7: now also U7.17 (2A0); no longer U9.17 (2A0), U9.2 (1A0)
- net SLV1C_MOSI: now also U7.3 (2Y0); no longer U9.18 (1Y0)
- net SLV1C_SCK: now also U9.18 (1Y0); no longer U7.3 (2Y0)
Changed lines of the file:
@@
 LIBS:valves
 LIBS:io_daughterboard-cache
-EELAYER 25 0
+EELAYER 26 0
 EELAYER END
 $Descr USLedger 17000 11000
@@
 F 0 "CON1" H 6900 7600 50  0000 C CNN
 F 1 "BARREL_JACK" H 6900 7150 50  0000 C CNN
-F 2 "Connect:BARREL_JACK" H 6900 7350 50  0001 C CNN
+F 2 "daughterfeet:BARREL_JACK" H 6900 7350 50  0001 C CNN
 F 3 "" H 6900 7350 50  0000 C CNN
 	1    6900 7350
@@
 F 0 "P3" H 1750 5850 50  0000 C CNN
 F 1 "Slave 1A" V 1850 5500 50  0000 C CNN
-F 2 "Connectors_Molex:Molex_PicoBlade_53047-0610_06x1.25mm_Straight" H 1750 5500 50  0001 C CNN
+F 2 "daughterfeet:Molex_PicoBlade_53047-0610_06x1.25mm_Straight" H 1750 5500 50  0001 C CNN
 F 3 "" H 1750 5500 50  0000 C CNN
 	1    1750 5500
@@
 	1    0    0    -1
 $EndComp
-Text Label 13750 2000 2    60   ~ 0
+Text Label 13750 5350 2    60   ~ 0
 SLV1C_SCK
 Text Label 13750 2100 2    60   ~ 0
@@
 Text Label 10400 1800 0    60   ~ 0
 SLV5C_MISO
-Text Label 10400 2000 0    60   ~ 0
+Text Label 10400 5350 0    60   ~ 0
 SPI1_SCK
 Text Label 10400 2100 0    60   ~ 0
@@
 	1    0    0    -1
 $EndComp
-Text Label 10400 5350 0    60   ~ 0
+Text Label 10400 2000 0    60   ~ 0
 SPI1_MOSI
 Text Label 10400 5450 0    60   ~ 0
@@
 Text Label 10400 6250 0    60   ~ 0
 SPI_D_~CS
-Text Label 13750 5350 2    60   ~ 0
+Text Label 13750 2000 2    60   ~ 0
 SLV1C_MOSI
 $Comp
@@
 F 0 "P7" H 3150 5850 50  0000 C CNN
 F 1 "Slave 1B" V 3250 5500 50  0000 C CNN
-F 2 "Connectors_Molex:Molex_PicoBlade_53047-0610_06x1.25mm_Straight" H 3150 5500 50  0001 C CNN
+F 2 "daughterfeet:Molex_PicoBlade_53047-0610_06x1.25mm_Straight" H 3150 5500 50  0001 C CNN
 F 3 "" H 3150 5500 50  0000 C CNN
 	1    3150 5500
@@
 F 0 "P11" H 4550 5850 50  0000 C CNN
 F 1 "Slave 1C" V 4650 5500 50  0000 C CNN
-F 2 "Connectors_Molex:Molex_PicoBlade_53047-0610_06x1.25mm_Straight" H 4550 5500 50  0001 C CNN
+F 2 "daughterfeet:Molex_PicoBlade_53047-0610_06x1.25mm_Straight" H 4550 5500 50  0001 C CNN
 F 3 "" H 4550 5500 50  0000 C CNN
 	1    4550 5500
@@
 F 0 "P4" H 1750 6850 50  0000 C CNN
 F 1 "Slave 3A" V 1850 6500 50  0000 C CNN
-F 2 "Connectors_Molex:Molex_PicoBlade_53047-0610_06x1.25mm_Straight" H 1750 6500 50  0001 C CNN
+F 2 "daughterfeet:Molex_PicoBlade_53047-0610_06x1.25mm_Straight" H 1750 6500 50  0001 C CNN
 F 3 "" H 1750 6500 50  0000 C CNN
 	1    1750 6500
@@
 F 0 "P8" H 3150 6850 50  0000 C CNN
 F 1 "Slave 3B" V 3250 6500 50  0000 C CNN
-F 2 "Connectors_Molex:Molex_PicoBlade_53047-0610_06x1.25mm_Straight" H 3150 6500 50  0001 C CNN
+F 2 "daughterfeet:Molex_PicoBlade_53047-0610_06x1.25mm_Straight" H 3150 6500 50  0001 C CNN
 F 3 "" H 3150 6500 50  0000 C CNN
 	1    3150 6500
@@
 F 0 "P12" H 4550 6850 50  0000 C CNN
 F 1 "Slave 3C" V 4650 6500 50  0000 C CNN
-F 2 "Connectors_Molex:Molex_PicoBlade_53047-0610_06x1.25mm_Straight" H 4550 6500 50  0001 C CNN
+F 2 "daughterfeet:Molex_PicoBlade_53047-0610_06x1.25mm_Straight" H 4550 6500 50  0001 C CNN
 F 3 "" H 4550 6500 50  0000 C CNN
 	1    4550 6500
@@
 F 0 "P15" H 5950 5850 50  0000 C CNN
 F 1 "Slave 1D" V 6050 5500 50  0000 C CNN
-F 2 "Connectors_Molex:Molex_PicoBlade_53047-0610_06x1.25mm_Straight" H 5950 5500 50  0001 C CNN
+F 2 "daughterfeet:Molex_PicoBlade_53047-0610_06x1.25mm_Straight" H 5950 5500 50  0001 C CNN
 F 3 "" H 5950 5500 50  0000 C CNN
 	1    5950 5500
@@
 F 0 "P16" H 5950 6850 50  0000 C CNN
 F 1 "Slave 3D" V 6050 6500 50  0000 C CNN
-F 2 "Connectors_Molex:Molex_PicoBlade_53047-0610_06x1.25mm_Straight" H 5950 6500 50  0001 C CNN
+F 2 "daughterfeet:Molex_PicoBlade_53047-0610_06x1.25mm_Straight" H 5950 6500 50  0001 C CNN
 F 3 "" H 5950 6500 50  0000 C CNN
 	1    5950 6500
@@
 F 0 "P5" H 1750 7850 50  0000 C CNN
 F 1 "Slave 4A" V 1850 7500 50  0000 C CNN
-F 2 "Connectors_Molex:Molex_PicoBlade_53047-0610_06x1.25mm_Straight" H 1750 7500 50  0001 C CNN
+F 2 "daughterfeet:Molex_PicoBlade_53047-0610_06x1.25mm_Straight" H 1750 7500 50  0001 C CNN
 F 3 "" H 1750 7500 50  0000 C CNN
 	1    1750 7500
@@
 F 0 "P9" H 3150 7850 50  0000 C CNN
 F 1 "Slave 4B" V 3250 7500 50  0000 C CNN
-F 2 "Connectors_Molex:Molex_PicoBlade_53047-0610_06x1.25mm_Straight" H 3150 7500 50  0001 C CNN
+F 2 "daughterfeet:Molex_PicoBlade_53047-0610_06x1.25mm_Straight" H 3150 7500 50  0001 C CNN
 F 3 "" H 3150 7500 50  0000 C CNN
 	1    3150 7500
@@
 F 0 "P13" H 4550 7850 50  0000 C CNN
 F 1 "Slave 4C" V 4650 7500 50  0000 C CNN
-F 2 "Connectors_Molex:Molex_PicoBlade_53047-0610_06x1.25mm_Straight" H 4550 7500 50  0001 C CNN
+F 2 "daughterfeet:Molex_PicoBlade_53047-0610_06x1.25mm_Straight" H 4550 7500 50  0001 C CNN
 F 3 "" H 4550 7500 50  0000 C CNN
 	1    4550 7500
@@
 F 0 "P6" H 1750 8850 50  0000 C CNN
 F 1 "Slave 5A" V 1850 8500 50  0000 C CNN
-F 2 "Connectors_Molex:Molex_PicoBlade_53047-0610_06x1.25mm_Straight" H 1750 8500 50  0001 C CNN
+F 2 "daughterfeet:Molex_PicoBlade_53047-0610_06x1.25mm_Straight" H 1750 8500 50  0001 C CNN
 F 3 "" H 1750 8500 50  0000 C CNN
 	1    1750 8500
@@
 F 0 "P10" H 3150 8850 50  0000 C CNN
 F 1 "Slave 5B" V 3250 8500 50  0000 C CNN
-F 2 "Connectors_Molex:Molex_PicoBlade_53047-0610_06x1.25mm_Straight" H 3150 8500 50  0001 C CNN
+F 2 "daughterfeet:Molex_PicoBlade_53047-0610_06x1.25mm_Straight" H 3150 8500 50  0001 C CNN
 F 3 "" H 3150 8500 50  0000 C CNN
 	1    3150 8500
@@
 F 0 "P14" H 4550 8850 50  0000 C CNN
 F 1 "Slave 5C" V 4650 8500 50  0000 C CNN
-F 2 "Connectors_Molex:Molex_PicoBlade_53047-0610_06x1.25mm_Straight" H 4550 8500 50  0001 C CNN
+F 2 "daughterfeet:Molex_PicoBlade_53047-0610_06x1.25mm_Straight" H 4550 8500 50  0001 C CNN
 F 3 "" H 4550 8500 50  0000 C CNN
 	1    4550 8500
@@
 F 0 "P17" H 5950 7850 50  0000 C CNN
 F 1 "Slave 4D" V 6050 7500 50  0000 C CNN
-F 2 "Connectors_Molex:Molex_PicoBlade_53047-0610_06x1.25mm_Straight" H 5950 7500 50  0001 C CNN
+F 2 "daughterfeet:Molex_PicoBlade_53047-0610_06x1.25mm_Straight" H 5950 7500 50  0001 C CNN
 F 3 "" H 5950 7500 50  0000 C CNN
 	1    5950 7500
@@
 F 0 "P18" H 5950 8850 50  0000 C CNN
 F 1 "Slave 5D" V 6050 8500 50  0000 C CNN
-F 2 "Connectors_Molex:Molex_PicoBlade_53047-0610_06x1.25mm_Straight" H 5950 8500 50  0001 C CNN
+F 2 "daughterfeet:Molex_PicoBlade_53047-0610_06x1.25mm_Straight" H 5950 8500 50  0001 C CNN
 F 3 "" H 5950 8500 50  0000 C CNN
 	1    5950 8500

Commit message: Fixed 3D models, made power traces heavier, pulled pour back from board edge
Connections:
- net PA5: now also U7.17 (2A0); no longer U9.17 (2A0), U9.2 (1A0)
- net PA7: now also U9.17 (2A0), U9.2 (1A0); no longer U7.17 (2A0)
- net SLV1C_MOSI: now also U9.18 (1Y0); no longer U7.3 (2Y0)
- net SLV1C_SCK: now also U7.3 (2Y0); no longer U9.18 (1Y0)
Changed lines of the file:
@@
 LIBS:valves
 LIBS:io_daughterboard-cache
-EELAYER 26 0
+EELAYER 25 0
 EELAYER END
 $Descr USLedger 17000 11000
@@
 	1    0    0    -1
 $EndComp
-Text Label 13750 5350 2    60   ~ 0
+Text Label 13750 2000 2    60   ~ 0
 SLV1C_SCK
 Text Label 13750 2100 2    60   ~ 0
@@
 Text Label 10400 1800 0    60   ~ 0
 SLV5C_MISO
-Text Label 10400 5350 0    60   ~ 0
+Text Label 10400 2000 0    60   ~ 0
 SPI1_SCK
 Text Label 10400 2100 0    60   ~ 0
@@
 	1    0    0    -1
 $EndComp
-Text Label 10400 2000 0    60   ~ 0
+Text Label 10400 5350 0    60   ~ 0
 SPI1_MOSI
 Text Label 10400 5450 0    60   ~ 0
@@
 Text Label 10400 6250 0    60   ~ 0
 SPI_D_~CS
-Text Label 13750 2000 2    60   ~ 0
+Text Label 13750 5350 2    60   ~ 0
 SLV1C_MOSI
 $Comp

Commit message: Changed LCD connector to Hirose FH12A.
Parts:
- LCD: renamed from J2; value 4-1734839-0 -> FH12A-40S-0.5SH; footprint daughterfeet:FPC_40 -> daughterfeet:FH12A-40S
- renumbered J1 to CTouch
Changed lines of the file:
@@
 $EndComp
 $Comp
-L XF2L-0625-1A J1
+L XF2L-0625-1A CTouch
 U 1 1 5825486E
 P 15750 1300
-F 0 "J1" H 15350 1400 60  0000 L CNN
+F 0 "CTouch" V 15300 1300 60  0000 R CNN
 F 1 "XF2L-0625-1A" H 15350 900 60  0000 L CNN
 F 2 "daughterfeet:XF2L-0625" H 15800 1400 60  0001 C CNN
@@
 $EndComp
 $Comp
-L 4-1734839-0 J2
+L 4-1734839-0 LCD
 U 1 1 58253EA8
 P 15800 4150
-F 0 "J2" H 13650 4300 60  0000 C CNN
-F 1 "4-1734839-0" H 13950 3800 60  0000 C CNN
-F 2 "daughterfeet:FPC_40" H 17050 4200 60  0001 C CNN
+F 0 "LCD" H 13650 4300 60  0000 C CNN
+F 1 "FH12A-40S-0.5SH" H 14050 3800 60  0000 C CNN
+F 2 "daughterfeet:FH12A-40S" H 17050 4200 60  0001 C CNN
 F 3 "" H 17050 4200 60  0001 C CNN
 	1    15800 4150
